File: ClockGen.kicad_sch (KiCad schematic)
At the start: 37 parts, among them Q10 KT315D, Q11 KT315D, Q5 KT315D, Q6 KT315D, U3 CD4017, Y1 4MHz

Commit message: Clock Gen Schematic Done
Parts:
- removed C? (x6): 100nF, Capacitor_THT:C_Disc_D5.0mm_W2.5mm_P2.50mm, symbol Device:C
- removed U? (x6): 4017, symbol 4xxx:4017
- added C10, C11, C12, C13, C14, C9: 100nF, Capacitor_THT:C_Disc_D5.0mm_W2.5mm_P2.50mm, symbol Device:C
- added U1, U2, U4, U5, U6, U7: CD4017, symbol 4xxx:4017
Connections:
- net CLK_4MHZ: now also U3.14 (CLK)
- net GND: now also C8.1, C10.1, C11.1, C12.1, C13.1, C14.1, C9.1, U1.13 (CKEN), U1.8 (VSS), U2.13 (CKEN), U2.8 (VSS), U4.13 (CKEN), U4.8 (VSS), U5.13 (CKEN), U5.8 (VSS), U6.13 (CKEN), U6.8 (VSS), U7.13 (CKEN), U7.8 (VSS); no longer C8.2
- net PBUS_12V: now also C8.2, U3.16 (VDD), C10.2, C11.2, C12.2, C13.2, C14.2, C9.2, U1.16 (VDD), U2.16 (VDD), U4.16 (VDD), U5.16 (VDD), U6.16 (VDD), U7.16 (VDD)
- net SIG_CLK_100HZ: now also U5.12 (Cout), U6.14 (CLK)
- net SIG_CLK_10HZ: now also U6.12 (Cout), U7.14 (CLK)
- net SIG_CLK_1HZ: now also U7.12 (Cout)
- net at U3.12 (Cout): now also U1.14 (CLK)
- removed net PBUS_12v: C8.1, U3.16 (VDD)
- new net: U5.10 (Q4), U5.15 (Reset)
- new net: U4.12 (Cout), U5.14 (CLK)
- new net: U2.10 (Q4), U2.15 (Reset)
- new net: U2.12 (Cout), U4.14 (CLK)
- new net: U1.12 (Cout), U2.14 (CLK)
- new net: U6.10 (Q4), U6.15 (Reset)
- new net: U7.10 (Q4), U7.15 (Reset)
- new net: U4.10 (Q4), U4.15 (Reset)
- new net: U1.10 (Q4), U1.15 (Reset)
- no-connect marks 69 -> 63
Other:
- note added: "Clock Divider"
- note removed: "Divider Board"
- moved on the sheet: C5, C6, C7, D4, D5, D?, Q10, Q11, Q5, Q6, Q?, R15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

Commit message: Started refactor of display section
Other:
- moved on the sheet: C5, C6, C7, D4, D5, D?, Q10, Q11, Q5, Q6, Q?, R15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

Commit message: Started PCB Outline & PSU
Other:
- moved on the sheet: U1, U2, U3, U4, U5, U6, U7
