File: DisplayControl.kicad_sch (KiCad schematic)
At the start: 187 parts

Commit message: Clock Gen Schematic Done
Connections:
- net at U?.12 (UG_C): now also D?.2 (A) (x5)
Changed lines of the file:
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@@
 	(title_block
 		(title "IV-6 VFD Clock")
-		(date "2025-06-22")
+		(date "2025-06-23")
 		(rev "MkII")
 		(company "ADBeta")

Commit message: Started refactor of display section
Connections:
- net at U?.12 (UG_C): now also D?.2 (A) (x5)
- net PBUS_20v renamed PBUS_20V
- net SIG_SEG_BUS_dp renamed SIG_SEG_BUS_P
- net VFD_SEG_dp renamed VFD_SEG_P
Other:
- note removed: "DONE"
- moved on the sheet: Q?, R?

Commit message: Started PCB Outline & PSU
Connections:
- net at U?.12 (UG_C): now also D?.2 (A) (x5)
Changed lines of the file:
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@@
 	(title_block
 		(title "IV-6 VFD Clock")
-		(date "2025-06-25")
+		(date "2025-07-01")
 		(rev "MkII")
 		(company "ADBeta")

Commit message: PSU Design started
Connections:
- net at U?.12 (UG_C): now also D?.2 (A) (x5)
Changed lines of the file:
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@@
 	(title_block
 		(title "IV-6 VFD Clock")
-		(date "2025-07-01")
+		(date "2025-07-06")
 		(rev "MkII")
 		(company "ADBeta")
