File: PowerControl.kicad_sch (KiCad schematic)
At the start: 40 parts, among them J1 INPUT_JACK, Q1 KT315D, Q13 KT315, Q2 KT315D, Q3 2n3906, Q4 2n3906, Q7 2n3904, Q8 2n3904, Q9 JE350

Commit message: Started PCB Outline & PSU
Other:
- note removed: "DONE"
- note removed: "Heater AC Frequency Generator"
- note removed: "Heater Filament H-Bridge Driver"
- note removed: "Main Power Regulation and Control"
- moved on the sheet: C1, C2, D2, D3, Q13, Q9, R1, R2, R23, R24, R?

Commit message: PSU Design started
Parts:
- added C15: 330pF, Capacitor_THT:C_Disc_D5.0mm_W2.5mm_P2.50mm, symbol Device:C
- added C16: 470uF, symbol Device:CP
- added D6: D_Schottky, symbol Device:D_Schottky
- added L1: L, symbol Device:L
- added R26: 10k, symbol Device:R
- added R27, R28: 180R, symbol Device:R
- added RV1: R_Potentiometer, symbol Device:R_Potentiometer
- added U8: MC33063AP, Package_DIP:DIP-8_W7.62mm, symbol Regulator_Switching:MC33063AP
Connections:
- net CTRL_DSP_EN: no longer R24.2
- net GND: now also C2.1; no longer C2.2
- net PBUS_EN_12v renamed PBUS_SW_12v
- net PBUS_EN_6v2 renamed PBUS_SW_6v
- net PBUS_SW_6v: now also C2.2; no longer C2.1
- net VFD_HTR_AC_A renamed VFD_HTR_SIG_A
- net VFD_HTR_AC_B renamed VFD_HTR_SIG_B
- new net: R26.1, R28.2, U8.5 (Vfb)
- new net: C15.1, U8.3 (TC)
- new net: D6.2 (A), U8.1 (SwC)
- new net: R27.2, U8.8 (DC)
- new net CTRL_SW_PWR: R24.2
Other:
- note added: "Input Power Control"
- note added: "TODO: BJT Switch timer circuit"
- note added: "VFD AC Oscillator"
- note added: "VFD H-Bridge"
- note removed: "Switched 12v output"
- note removed: "Switched 6.2v output (for VFD heater)"
- moved on the sheet: 100nF, C1, C2, C3, C4, C?, D1, D2, D3, J1, Q1, Q13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

Commit message: PSU Schematic Finished
Parts:
- L1: value L -> 100uH
- R26: value 10k -> 1K
- R28: value 180R -> 10K
- RV1: value R_Potentiometer -> 470R
Connections:
- net GND: now also C15.2, C16.2, R26.1, U8.2 (SwE), U8.4 (GND)
- net PBUS_SW_12v: now also L1.2, R27.1, U8.6 (Vin), U8.7 (Ipk)
- net at RV1.1: now also R28.1, U8.5 (Vfb)
- net at RV1.2: now also R26.2
- net at L1.1: now also D6.2 (A), U8.1 (SwC)
- net at D6.1 (K): now also C16.1, R28.2
- no-connect marks 0 -> 1
Other:
- note added: "25V PSU"
- moved on the sheet: C15, C16, C3, C4, D6, L1, Q1, Q2, Q3, Q4, Q7, Q8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
